Commit message: Gazebo and Moveit fully synched but mimic not yet

File: franka_panda/description/panda.urdf (robot description, URDF)
Before this commit: robot panda, 13 links, 12 joints
Joints:
- joint panda_finger_joint2: mimic (none) -> joint=panda_finger_joint1 multiplier=1.0 offset=0.0

File: panda_moveit_config/config/panda.gazebo.xacro (robot description, xacro)
@@ -4,5 +4,5 @@
   <gazebo>
     <plugin filename="gz_ros2_control-system" name="gz_ros2_control::GazeboSimROS2ControlPlugin">
-      <parameters>$(find panda_moveit_config)/config/moveit_controllers.yaml</parameters>
+      <parameters>$(find panda_moveit_config)/config/gazebo_controllers.yaml</parameters>
     </plugin>
   </gazebo>

File: panda_moveit_config/config/panda.urdf.xacro (robot description, xacro)
@@ -8,5 +8,5 @@
     <xacro:include filename="panda.gazebo.xacro" />
     <!-- 1. Call the control macro (Ensure this hardware is set to GazeboSimSystem) -->
-    <xacro:panda_ros2_control name="PandaGazeboClassicSystem" initial_positions_file="$(arg initial_positions_file)"/>
+    <xacro:panda_ros2_control name="PandaIgnitionSystem" initial_positions_file="$(arg initial_positions_file)"/>
     <!-- 2. Call the gazebo macro we fixed above -->
     <xacro:panda_gazebo />

Commit message: The gripper opens both fingers but used Follow Trajectory

File: franka_panda/description/panda.urdf (robot description, URDF)
Before this commit: robot panda, 13 links, 12 joints
Joints:
- joint panda_finger_joint2: mimic joint=panda_finger_joint1 multiplier=1.0 offset=0.0 -> (none)

File: panda_moveit_config/config/panda.gazebo.xacro (robot description, xacro)
@@ -59,11 +59,11 @@
   </gazebo>
   <gazebo reference="panda_leftfinger">
-    <mu1>0.2</mu1>
-    <mu2>0.2</mu2>
+    <mu1>1.1</mu1>
+    <mu2>1.1</mu2>
     <self_collide>true</self_collide>
   </gazebo>
   <gazebo reference="panda_rightfinger">
-    <mu1>0.2</mu1>
-    <mu2>0.2</mu2>
+    <mu1>1.1</mu1>
+    <mu2>1.1</mu2>
     <self_collide>true</self_collide>
   </gazebo>
